File: reef-piHat.kicad_pcb (KiCad board)
At the start: 2 copper layers, 65 x 56 mm, 35 parts, among them J1 Doser, J10 ATO2, J11 ph1, J12 ph2, J13 5vPower, J14 Temp1, J15 Temp2, J16 Temp3, J2 Light1, J3 40HAT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

Commit message: Complete layout and update gerbers
Routing:
- net /P5V_HAT: track 73.6 -> 74.3 mm
Other:
- board text removed: "If you want to use an SMT 40-pin header, please move the top edge up by 0.5mm and locate the header in the same location as the current TH part."
- board text removed: "This is a HAT compatible PCB starting design based on the official Raspberry Pi specs at: https://github.com/raspberrypi/hats/blob/master/designguide.md Currently the camera slot and display cutout are not here. See the schematic for the details on the EEPROM and power setup. This board does have the correct components for powering the Pi via the HAT. If you need the Pi to provide 5V or 3.3V, ple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"
Changed lines of the file:
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@@
   (general
     (thickness 1.6)
-    (drawings 61)
-    (tracks 420)
+    (drawings 59)
+    (tracks 421)
     (zones 0)
     (modules 35)
@@
     (tags "SOIC 1.27")
     (attr smd)
-    (fp_text reference U2 (at 0 -3.5 180) (layer F.SilkS)
-      (effects (font (size 1 1) (thickness 0.15)))
-    )
-    (fp_text value CAT24C32 (at 0 3.5 180) (layer F.Fab)
+    (fp_text reference U2 (at 0 0 180) (layer F.SilkS)
+      (effects (font (size 1 1) (thickness 0.15)))
+    )
+    (fp_text value CAT24C32 (at 0 3.5 180) (layer F.SilkS)
       (effects (font (size 1 1) (thickness 0.15)))
     )
@@
     (tags "resistor handsolder")
     (attr smd)
-    (fp_text reference R1 (at 0 -1.43) (layer F.SilkS)
-      (effects (font (size 1 1) (thickness 0.15)))
-    )
-    (fp_text value DNP (at 0 1.43) (layer F.Fab)
+    (fp_text reference R1 (at -2.681 0.0635) (layer F.SilkS)
+      (effects (font (size 1 1) (thickness 0.15)))
+    )
+    (fp_text value DNP (at 3.2245 0.0635) (layer F.SilkS)
       (effects (font (size 1 1) (thickness 0.15)))
     )
@@
     (tags "resistor handsolder")
     (attr smd)
-    (fp_text reference R2 (at 0 -1.43) (layer F.SilkS)
-      (effects (font (size 1 1) (thickness 0.15)))
-    )
-    (fp_text value 10K (at 0 1.43) (layer F.Fab)
+    (fp_text reference R2 (at -2.653 0.0635) (layer F.SilkS)
+      (effects (font (size 1 1) (thickness 0.15)))
+    )
+    (fp_text value 10K (at -5.701 0.0635) (layer F.SilkS)
       (effects (font (size 1 1) (thickness 0.15)))
     )
@@
     (tags "resistor handsolder")
     (attr smd)
-    (fp_text reference R3 (at 0 -1.43) (layer F.SilkS)
-      (effects (font (size 1 1) (thickness 0.15)))
-    )
-    (fp_text value 3.9K (at 0 1.43) (layer F.Fab)
+    (fp_text reference R3 (at -2.667 0) (layer F.SilkS)
+      (effects (font (size 1 1) (thickness 0.15)))
+    )
+    (fp_text value 3.9K (at -5.9055 0) (layer F.SilkS)
       (effects (font (size 1 1) (thickness 0.15)))
     )
@@
     (tags "resistor handsolder")
     (attr smd)
-    (fp_text reference R4 (at 0 -1.43) (layer F.SilkS)
-      (effects (font (size 1 1) (thickness 0.15)))
-    )
-    (fp_text value 3.9K (at 0 1.43) (layer F.Fab)
+    (fp_text reference R4 (at -2.667 -0.0635) (layer F.SilkS)
+      (effects (font (size 1 1) (thickness 0.15)))
+    )
+    (fp_text value 3.9K (at -5.9055 -0.0635) (layer F.SilkS)
       (effects (font (size 1 1) (thickness 0.15)))
     )
@@
   )
   (gr_text + (at 125.095 112.8395) (layer F.SilkS)
-    (effects (font (size 1.5 1.5) (thickness 0.3)))
-  )
-  (gr_text "If you want to use an SMT 40-pin header, please move the top edge up \nby 0.5mm and locate the header in the same location as the current TH part." (at 117.3 47.5) (layer Cmts.User)
-    (effects (font (size 1.5 1.5) (thickness 0.3)))
-  )
-  (gr_text "This is a HAT compatible PCB starting design based on the official\nRaspberry Pi specs at:\nhttps://github.com/raspberrypi/hats/blob/master/designguide.md\n\nCurrently the camera slot and display cutout are not here. \nSee the schematic for the details on the EEPROM and power setup.\n\nThis board does have the correct components for powering the Pi via\nthe HAT. If you need the Pi to provide 5V or 3.3V, please remove or\nconnect the appropriate components." (at 189.4 83.7) (layer Cmts.User)
     (effects (font (size 1.5 1.5) (thickness 0.3)))
   )
@@
   (segment (start 91.7575 75.692) (end 91.7575 78.9305) (width 0.25) (layer F.Cu) (net 5))
   (segment (start 91.567 79.121) (end 91.567 86.1695) (width 0.25) (layer F.Cu) (net 5))
-  (segment (start 89.46 63.05) (end 86.92 63.05) (width 0.4) (layer F.Cu) (net 59))
   (segment (start 106.8705 115.316) (end 87.249 115.316) (width 0.4) (layer F.Cu) (net 5))
   (segment (start 87.249 115.316) (end 85.598 113.665) (width 0.4) (layer F.Cu) (net 5))
@@
   (segment (start 124.46 103.8225) (end 127.5715 103.8225) (width 0.15) (layer F.Cu) (net 57))
   (segment (start 123.5075 102.87) (end 124.46 103.8225) (width 0.15) (layer F.Cu) (net 57))
+  (segment (start 89.46 63.05) (end 86.92 63.05) (width 0.4) (layer F.Cu) (net 59))
   (segment (start 108.7285 108.077) (end 110.744 108.077) (width 0.2) (layer F.Cu) (net 59))
   (segment (start 110.744 108.077) (end 110.744 108.077) (width 0.2) (layer F.Cu) (net 59))
@@
   (segment (start 110.744 103.505) (end 108.881 103.505) (width 0.2) (layer F.Cu) (net 59))
   (segment (start 86.92 63.05) (end 86.1115 63.05) (width 0.25) (layer B.Cu) (net 59))
-  (segment (start 86.1115 63.05) (end 85.0265 64.135) (width 0.25) (layer B.Cu) (net 59))
-  (segment (start 85.0265 64.135) (end 85.0265 69.469) (width 0.25) (layer B.Cu) (net 59))
-  (segment (start 85.0265 69.469) (end 89.5985 74.041) (width 0.25) (layer B.Cu) (net 59))
   (segment (start 89.5985 74.041) (end 107.061 74.041) (width 0.25) (layer B.Cu) (net 59))
   (segment (start 110.744 77.724) (end 110.744 103.505) (width 0.25) (layer B.Cu) (net 59))
   (segment (start 107.061 74.041) (end 110.744 77.724) (width 0.25) (layer B.Cu) (net 59))
+  (segment (start 86.92 63.05) (end 85.921 63.05) (width 0.15) (layer B.Cu) (net 59))
+  (segment (start 85.2805 63.6905) (end 85.2805 69.723) (width 0.25) (layer B.Cu) (net 59))
+  (segment (start 85.921 63.05) (end 85.2805 63.6905) (width 0.25) (layer B.Cu) (net 59))
+  (segment (start 85.2805 69.723) (end 89.5985 74.041) (width 0.25) (layer B.Cu) (net 59))
   (segment (start 106.0285 107.127) (end 106.0285 108.077) (width 0.2) (layer F.Cu) (net 60))
   (segment (start 106.0285 109.027) (end 106.0285 108.077) (width 0.2) (layer F.Cu) (net 60))
   (segment (start 106.0285 110.9155) (end 105.9815 110.9625) (width 0.2) (layer F.Cu) (net 60))
   (segment (start 106.0285 109.027) (end 106.0285 110.9155) (width 0.2) (layer F.Cu) (net 60))
+  (segment (start 120.9395 73.9775) (end 120.495 74.422) (width 0.15) (layer F.Cu) (net 61))
+  (segment (start 122.9665 73.9775) (end 120.9395 73.9775) (width 0.15) (layer F.Cu) (net 61))
+  (segment (start 124.8055 77.216) (end 124.8055 74.6405) (width 0.15) (layer F.Cu) (net 61))
+  (segment (start 124.1425 73.9775) (end 122.9665 73.9775) (width 0.15) (layer F.Cu) (net 61))
+  (segment (start 124.8055 74.6405) (end 124.1425 73.9775) (width 0.15) (layer F.Cu) (net 61))
   (segment (start 107.24 65.59) (end 107.24 67.616) (width 0.15) (layer B.Cu) (net 62))
   (segment (start 107.24 67.616) (end 108.712 69.088) (width 0.15) (layer B.Cu) (net 62))
@@
   (segment (start 118.618 69.088) (end 118.618 69.088) (width 0.15) (layer B.Cu) (net 62))
   (via (at 118.618 69.088) (size 0.6) (drill 0.2) (layers F.Cu B.Cu) (net 62))
-  (segment (start 120.9395 73.9775) (end 120.495 74.422) (width 0.15) (layer F.Cu) (net 61))
-  (segment (start 122.9665 73.9775) (end 120.9395 73.9775) (width 0.15) (layer F.Cu) (net 61))
-  (segment (start 124.8055 77.216) (end 124.8055 74.6405) (width 0.15) (layer F.Cu) (net 61))
-  (segment (start 124.1425 73.9775) (end 122.9665 73.9775) (width 0.15) (layer F.Cu) (net 61))
-  (segment (start 124.8055 74.6405) (end 124.1425 73.9775) (width 0.15) (layer F.Cu) (net 61))
   (segment (start 122.9665 75.2475) (end 122.2375 75.2475) (width 0.15) (layer F.Cu) (net 62))
   (segment (start 122.2375 75.2475) (end 121.4755 76.0095) (width 0.15) (layer F.Cu) (net 62))

Commit message: Add readme and images
Parts:
- C1: value 10uF -> 1uF
Changed lines of the file:
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@@
   (general
     (thickness 1.6)
-    (drawings 59)
+    (drawings 61)
     (tracks 421)
     (zones 0)
@@
       (effects (font (size 1 1) (thickness 0.15)))
     )
-    (fp_text value 10uF (at 3.0115 -1.778) (layer F.SilkS)
+    (fp_text value 1uF (at 3.0115 -1.778) (layer F.SilkS)
       (effects (font (size 1 1) (thickness 0.15)))
     )
@@
     )
   )
+  (gr_circle (center 105.6005 106.045) (end 105.8545 106.299) (layer F.SilkS) (width 0.15))
+  (gr_circle (center 126.8095 75.2475) (end 127.0635 75.5015) (layer F.SilkS) (width 0.15))
   (gr_text "reef-pi hat\ngithub.com/ranthalion/reef-piHat" (at 134.366 77.724) (layer B.SilkS)
     (effects (font (size 0.8 0.8) (thickness 0.2)) (justify left mirror))
