File: reef-piHat.sch (KiCad schematic (older format))
At the start: 33 parts, among them J1 Doser, J10 ATO2, J11 ph1, J12 ph2, J13 5vPower, J14 Temp1, J15 Temp2, J16 Temp3, J2 Light1, J3 40HAT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

Commit message: Add readme and images
Other:
- moved on the sheet: J11, J12, J13, J14, J15, J16, J5, J6, J7, R13, U3
