File: v2/reef-piHat.sch (KiCad schematic (older format))
At the start: 53 parts, among them J1 Doser, J10 ATO2, J11 ph1, J12 ph2, J13 5vPower, J14 Temp1, J15 Temp2, J16 Temp3, J2 Light1, J3 40HAT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

Commit message: Gerbers
Parts:
- added R3: 220, Resistor_SMD:R_0603_1608Metric_Pad1.05x0.95mm_HandSolder, symbol pspice:R
- C1: value 10uF -> 1uF
- D1, D10, D2, D3, D4, D5, D6, D7, D8, D9: value ZMMxx -> z3.3
- R1, R2: value R -> 220
Connections:
- net A4: now also RN1.6 (R3.2); no longer RN1.5 (R4.2)
- net A5: now also RN1.7 (R2.2); no longer RN1.6 (R3.2)
- net GND: now also RN1.1 (R1.1); no longer RN1.4 (R4.1)
- net LED15: now also R3.1; no longer RN1.8 (R1.2)
- net at J2.1 (Pin_1): now also R3.2; no longer RN1.1 (R1.1)
- net OE: now reaches U1.23 (~OE)
- net OE: now also RN1.8 (R1.2); no longer RN1.7 (R2.2)
Other:
- moved on the sheet: D2, J13, J2, J5, J8, R1, RN1

Commit message: update images
Connections:
- no-connect marks 15 -> 17
Other:
- note added: "1 Wire Headers"
- note added: "ATO Headers"
- note added: "I2C Headers"
- note added: "PWM Output"
- note added: "Protected GPIO Header"
- note added: "ULN2803 Output"
- moved on the sheet: A0, A1, A2, A3, A4, A5, C1, D1, D10, D2, D3, D4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
