File: v2/reef-piHat.kicad_pcb (KiCad board)
At the start: 2 copper layers, 65 x 56 mm, 55 parts, among them J1 Doser, J10 ATO2, J11 ph1, J12 ph2, J13 5vPower, J14 Temp1, J15 Temp2, J16 Temp3, J2 Light1, J3 40HAT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

Commit message: Gerbers
Parts:
- added R3: 220, Resistor_SMD:R_0603_1608Metric_Pad1.05x0.95mm_HandSolder, F.Cu at (97.9, 104.1)
- D1, D10, D2, D3, D4, D5, D6, D7, D8, D9: value ZMMxx -> z3.3
- R1, R2: value R -> 220
- REF**: value OSHW-Logo2_7.3x6mm_SilkScreen -> logo
- moved R7 20.0 mm to (112.8, 114.2), turned to 0 degrees
- moved G*** 20.0 mm to (138.0, 103.2), turned to 90 degrees
- moved R6 17.3 mm to (112.8, 111.5)
- moved Q2 15.6 mm to (104.9, 112.6), turned to 90 degrees
- moved Q1 13.4 mm to (109.0, 112.8), turned to 270 degrees
- moved RN1 1.63 mm to (97.8, 106.9)
- moved RN7 1.41 mm to (135.0, 71.5)
Connections:
- RN1 pad 1: Net-(J2-Pad1) -> GND
- RN1 pad 4: GND -> Net-(RN1-Pad4)
- RN1 pad 5: /A4 -> Net-(RN1-Pad5)
- RN1 pad 6: /A5 -> /A4
- RN1 pad 7: Net-(RN1-Pad7) -> /A5
- RN1 pad 8: /LED15 -> /OE
- U1 pad 23: Net-(RN1-Pad7) -> /OE
Routing:
- net /P5V_HAT: track 171.3 -> 186.4 mm
- net /OE: track 0.00 -> 6.16 mm
- net Net-(RN1-Pad7): track 5.82 -> 0.00 mm
- net GND: track 13.5 -> 17.2 mm
- net /PB5: track 30.8 -> 28.2 mm
- net /PB3: track 22.2 -> 20.0 mm
- net /PB4: track 22.5 -> 20.3 mm
- net /PB6: track 29.4 -> 27.4 mm
- net Net-(Q1-Pad4): track 5.88 -> 7.67 mm
- net Net-(J7-Pad7): track 7.34 -> 8.75 mm
- net Net-(J7-Pad8): track 5.76 -> 7.17 mm
- net Net-(J7-Pad9): track 4.41 -> 5.82 mm
- net /PB7: track 31.0 -> 29.8 mm
- net Net-(J2-Pad1): track 6.18 -> 7.24 mm
- net /PB1: track 17.5 -> 16.6 mm
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Other:
- board text added: "PCA9685 Address"

Commit message: Update gerbers
Parts:
- C1: value 10uF -> 1uF; footprint Capacitor_SMD:C_1206_3216Metric_Pad1.42x1.75mm_HandSolder -> Capacitor_SMD:C_0603_1608Metric_Pad1.05x0.95mm_HandSolder
- D1, D10, D2, D3, D4, D5, D6, D7, D8, D9, R1, R13, R2, R6, R7: moved to F.Cu
- J13, J5: footprint Connector_PinHeader_2.54mm:PinHeader_1x02_P2.54mm_Vertical -> Connector_JST:JST_XH_B02B-XH-A_1x02_P2.50mm_Vertical
- Q1: footprint Package_TO_SOT_SMD:SOT-23-6_Handsoldering -> Package_TO_SOT_SMD:SOT-23-6; moved to F.Cu
- Q2: footprint Package_TO_SOT_SMD:SOT-23_Handsoldering -> Package_TO_SOT_SMD:SOT-23; moved to F.Cu
- moved REF** 22.4 mm to (117.7, 99.1)
- moved U3 12.2 mm to (129.4, 101.1), turned to 0 degrees
- moved R2 11.1 mm to (94.8, 84.8), turned to 90 degrees
- moved J6 10.9 mm to (138.4, 98.3)
- moved R1 10.1 mm to (94.8, 75.5), turned to 90 degrees
- moved Q2 7.62 mm to (97.3, 113.6), turned to 180 degrees
- moved C1 7.32 mm to (106.6, 110.2), turned to 0 degrees
- moved R6 6.94 mm to (106.6, 114.7)
- moved R7 6.55 mm to (106.6, 111.9)
- moved A0 6.41 mm to (125.6, 113.3)
- moved A1 6.41 mm to (123.0, 113.3)
- moved A2 6.41 mm to (120.4, 113.3)
- moved A3 6.41 mm to (117.8, 113.3)
- moved A4 6.41 mm to (115.2, 113.3)
- moved A5 6.41 mm to (112.6, 113.3)
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Connections:
- net Net-(J6-Pad4) renamed /PA_O3
- net Net-(J6-Pad7) renamed /PA_O8
- J13 pad 1: /P5V -> GND
- J13 pad 2: GND -> /P5V
- J6 pad 1: Net-(J6-Pad1) -> /PA_O2
- J6 pad 2: Net-(J6-Pad2) -> /PA_O1
- J6 pad 3: Net-(J6-Pad3) -> /PA_O4
- J6 pad 5: Net-(J6-Pad5) -> /PA_O6
- J6 pad 6: Net-(J6-Pad6) -> /PA_O5
- J6 pad 8: Net-(J6-Pad8) -> /PA_O7
- U3 pad 12: Net-(J6-Pad5) -> /PA_O7
- U3 pad 13: Net-(J6-Pad3) -> /PA_O6
- U3 pad 14: Net-(J6-Pad1) -> /PA_O5
- U3 pad 15: Net-(J6-Pad2) -> /PA_O4
- U3 pad 17: Net-(J6-Pad6) -> /PA_O2
- U3 pad 18: Net-(J6-Pad8) -> /PA_O1
Routing:
- net /P5V_HAT: track 186.4 -> 166.1 mm, vias 3 -> 1
- net /PA8: track 35.1 -> 51.4 mm
- net Net-(J6-Pad8): track 15.3 -> 0.00 mm
- net /PA7: track 38.2 -> 52.8 mm
- net Net-(J6-Pad5): track 13.6 -> 0.00 mm
- net /1WIRE: track 61.5 -> 48.6 mm
- net /PA6: track 37.6 -> 50.5 mm
- net Net-(J6-Pad6): track 12.2 -> 0.00 mm
- net /PA5: track 33.9 -> 46.1 mm
- net GND: track 17.2 -> 5.00 mm, vias 0 -> 1
- net Net-(J6-Pad3): track 11.5 -> 0.00 mm
- net /PA4: track 36.4 -> 47.8 mm
- net /PA_O8: track 16.5 -> 5.08 mm
- net /P5V: track 27.8 -> 16.9 mm
- net /PA3: track 32.7 -> 43.2 mm
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Other:
- board text added: "reef-pi hat (goby) github.com/ranthalion/reef-piHat"
- board text removed: "reef-pi hat v2 github.com/ranthalion/reef-piHat"
