File: v3/reef-piHat.kicad_pcb (KiCad board)
At the start: 2 copper layers, 65 x 56 mm, 116 parts, among them J1 Doser, J10 ATO2, J11 I2C, J12 I2C, J13 5vPower, J14 Temp1, J15 Temp2, J16 Temp3, J2 Light1, J3 40HAT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

Commit message: Update gerbers
Parts:
- REF**: value OSHW-Logo2_7.3x6mm_SilkScreen -> OSHW-Logo
Changed lines of the file:
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@@
       (effects (font (size 1 1) (thickness 0.15)))
     )
-    (fp_text value OSHW-Logo2_7.3x6mm_SilkScreen (at 0.75 0) (layer F.Fab) hide
+    (fp_text value OSHW-Logo (at 0.75 0) (layer F.Fab) hide
       (effects (font (size 1 1) (thickness 0.15)))
     )
